Commit message: use the urdf in robot_arm

File: robot_arm/urdf/wx250s.urdf (robot description, URDF)
Before this commit: robot wx250s, 14 links, 13 joints
Links:
- link wx250s/base_link: geometry collision mesh filename=package://robot_arm/meshes/base.stl scale=0.001 0.001 0.001; visual mesh filename=package://robot_arm/meshes/base.stl scale=0.001 0.001 0.001
- link wx250s/gripper_bar_link: geometry collision mesh filename=package://robot_arm/meshes/gripper_bar.stl scale=0.001 0.001 0.001; visual mesh filename=package://robot_arm/meshes/gripper_bar.stl scale=0.001 0.001 0.001
- link wx250s/gripper_link: geometry collision mesh filename=package://robot_arm/meshes/gripper.stl scale=0.001 0.001 0.001; visual mesh filename=package://robot_arm/meshes/gripper.stl scale=0.001 0.001 0.001
- link wx250s/gripper_prop_link: geometry collision mesh filename=package://robot_arm/meshes/gripper_prop.stl scale=0.001 0.001 0.001; visual mesh filename=package://robot_arm/meshes/gripper_prop.stl scale=0.001 0.001 0.001
- link wx250s/left_finger_link: geometry collision mesh filename=package://robot_arm/meshes/gripper_finger.stl scale=0.001 0.001 0.001; visual mesh filename=package://robot_arm/meshes/gripper_finger.stl scale=0.001 0.001 0.001
- link wx250s/lower_forearm_link: geometry collision mesh filename=package://robot_arm/meshes/lower_forearm.stl scale=0.001 0.001 0.001; visual mesh filename=package://robot_arm/meshes/lower_forearm.stl scale=0.001 0.001 0.001
- link wx250s/right_finger_link: geometry collision mesh filename=package://robot_arm/meshes/gripper_finger.stl scale=0.001 0.001 0.001; visual mesh filename=package://robot_arm/meshes/gripper_finger.stl scale=0.001 0.001 0.001
- link wx250s/shoulder_link: geometry collision mesh filename=package://robot_arm/meshes/shoulder.stl scale=0.001 0.001 0.001; visual mesh filename=package://robot_arm/meshes/shoulder.stl scale=0.001 0.001 0.001
- link wx250s/upper_arm_link: geometry collision mesh filename=package://robot_arm/meshes/upper_arm.stl scale=0.001 0.001 0.001; visual mesh filename=package://robot_arm/meshes/upper_arm.stl scale=0.001 0.001 0.001
- link wx250s/upper_forearm_link: geometry collision mesh filename=package://robot_arm/meshes/upper_forearm.stl scale=0.001 0.001 0.001; visual mesh filename=package://robot_arm/meshes/upper_forearm.stl scale=0.001 0.001 0.001
- link wx250s/wrist_link: geometry collision mesh filename=package://robot_arm/meshes/wrist.stl scale=0.001 0.001 0.001; visual mesh filename=package://robot_arm/meshes/wrist.stl scale=0.001 0.001 0.001
Joints:
- joint elbow: limit lower=-2.14675 upper=1.60570 effort=15 velocity=3.14159 -> lower=-2.1467549799530254 upper=1.6057029118347832 effort=15 velocity=3.141592653589793
- joint forearm_roll: limit lower=-3.14158 upper=3.14158 effort=2 velocity=3.14159 -> lower=-3.141582653589793 upper=3.141582653589793 effort=2 velocity=3.141592653589793
- joint gripper: limit effort=1 velocity=3.14159 -> effort=1 velocity=3.141592653589793; type revolute -> continuous
- joint left_finger: mimic joint=gripper multiplier=-1.0 offset=0.015 -> (none)
- joint right_finger: mimic joint=left_finger multiplier=-1 offset=0 -> (none)
- joint shoulder: limit lower=-1.88496 upper=1.98968 effort=20 velocity=3.14159 -> lower=-1.8849555921538759 upper=1.9896753472735358 effort=20 velocity=3.141592653589793
- joint waist: limit lower=-3.14158 upper=3.14158 effort=10 velocity=3.14159 -> lower=-3.141582653589793 upper=3.141582653589793 effort=10 velocity=3.141592653589793
- joint wrist_angle: limit lower=-1.74533 upper=2.14675 effort=5 velocity=3.14159 -> lower=-1.7453292519943295 upper=2.1467549799530254 effort=5 velocity=3.141592653589793
- joint wrist_rotate: limit lower=-3.14158 upper=3.14158 effort=1 velocity=3.14159 -> lower=-3.141582653589793 upper=3.141582653589793 effort=1 velocity=3.141592653589793
